Commit message: Add lidar and rviz visualization

File: ros2_ws/src/hardware/justina_description/urdf/justina_base.xacro (robot description, xacro)
@@ -28,4 +28,10 @@
     <xacro:property name="caster_inertia_y" value="${2.0/5.0 * caster_mass * caster_radius * caster_radius}"/>
     <xacro:property name="caster_inertia_z" value="${2.0/5.0 * caster_mass * caster_radius * caster_radius}"/>
+    <xacro:property name="laser_radius" value="0.06"/>
+    <xacro:property name="laser_height" value="0.05"/>
+    <xacro:property name="laser_mass" value="0.2"/>
+    <xacro:property name="laser_inertia_xx" value="${(1/12) * laser_mass * (3*laser_radius*laser_radius + laser_height*laser_height)}"/>
+    <xacro:property name="laser_inertia_yy" value="${(1/12) * laser_mass * (3*laser_radius*laser_radius + laser_height*laser_height)}"/>
+    <xacro:property name="laser_inertia_zz" value="${(1/2) * laser_mass * laser_radius*laser_radius}"/>
     <!-- Control Parameters -->
     <xacro:property name="max_linear_acceleration" value="10"/>
@@ -123,4 +129,26 @@
         </inertial>
     </link>
+    <link name="laser_link">
+      <visual>
+         <origin xyz="0 0 0"/>
+         <geometry>
+            <cylinder length="${laser_height}" radius="${laser_radius}"/>
+         </geometry>
+         <material name="laser_material">
+            <color rgba="0.07 0.07 0.07 1.0"/>
+         </material>
+      </visual>
+      <collision>
+         <origin xyz="0 0 0"/>
+         <geometry>
+            <cylinder length="${laser_height}" radius="${laser_radius}"/>
+         </geometry>
+      </collision>
+      <inertial>
+        <mass value="${laser_mass}"/>
+        <inertia ixx="${laser_inertia_xx}" ixy="0.0" ixz="0.0" iyy="${laser_inertia_yy}" iyz="0" izz="${laser_inertia_zz}"/>
+        <origin xyz="0 0 0" rpy="0 0 0"/>
+      </inertial>
+   </link>
     <!-- Joints -->
     <!-- Left Wheel Joint -->
@@ -148,4 +176,10 @@
         <child link="caster_link"/>
     </joint>
+    <!-- Body to laser joint -->
+    <joint name="laser_joint" type="fixed">
+      <origin xyz="${body_length/2 - laser_radius} 0.0 ${body_height/2+laser_height/2}" rpy="0 0 0"/>
+      <parent link="body_link"/>
+      <child link="laser_link"/>
+    </joint>
     <!-- Gazebo Parameters -->
     <gazebo reference="body_link">
@@ -164,4 +198,8 @@
         <mu1>0.000001</mu1>
         <mu2>0.000001</mu2>
+    </gazebo>
+    <gazebo reference="laser_link">
+        <mu1>1.0</mu1>
+        <mu2>1.0</mu2>
     </gazebo>
     <!-- Gazebo Plugins -->
@@ -183,3 +221,31 @@
         </plugin>
     </gazebo>
+    <gazebo reference="laser_link">
+      <sensor name="laser" type="gpu_lidar">
+         <pose> 0 0 0 0 0 0 </pose>
+         <always_on>true</always_on>
+         <visualize>true</visualize>
+         <update_rate>10</update_rate>
+         <topic>scan</topic>
+         <gz_frame_id>laser_link</gz_frame_id>
+         <lidar>
+           <scan>
+             <horizontal>
+               <samples>480</samples>
+               <min_angle>-2.0944</min_angle>
+               <max_angle>2.0944</max_angle>
+             </horizontal>
+           </scan>
+           <range>
+             <min>0.1</min>
+             <max>10.0</max>
+           </range>
+           <noise>
+             <type>gaussian</type>
+             <mean>0.0</mean>
+             <stddev>0.03</stddev>
+           </noise>
+         </lidar>
+      </sensor>
+    </gazebo>
 </robot>

Commit message: Reorder justina_gui, add simple move pakage

File: ros2_ws/src/hardware/justina_description/urdf/justina_base.xacro (robot description, xacro)
@@ -37,5 +37,5 @@
     <xacro:property name="max_linear_acceleration" value="10"/>
     <!-- Links -->
-    <link name="base_footprint"/>
+    <link name="base_link"/>
     <!-- Body Link -->
     <link name="body_link">
@@ -155,5 +155,5 @@
    <joint name="base_to_body" type="fixed">
      <origin xyz="0 0 ${body_height/2}" rpy="0 0 0"/>
-     <parent link="base_footprint"/>
+     <parent link="base_link"/>
      <child link="body_link"/>
    </joint>
@@ -221,5 +221,5 @@
         <tf_topic>tf</tf_topic>
         <frame_id>/odom</frame_id>
-        <child_frame_id>/base_footprint</child_frame_id>
+        <child_frame_id>/base_link</child_frame_id>
         <odom_topic>odom</odom_topic>
       </plugin>
@@ -253,5 +253,5 @@
              <type>gaussian</type>
              <mean>0.0</mean>
-             <stddev>0.03</stddev>
+             <stddev>0.02</stddev>
            </noise>
          </lidar>
