Commit message: Working base with xarm. No cameras, lidar nor other sensor. No control for xarm

File: ros2_ws/src/hardware/justina_description/urdf/justina.xacro (robot description, xacro)
@@ -2,4 +2,10 @@
 <robot name="justina" xmlns:xacro="http://www.ros.org/wiki/xacro">
   <xacro:include filename="$(find justina_description)/urdf/justina_base.xacro"/>
-  <!-- <xacro:include filename="$(find xarm_description)/urdf/xarm_device.urdf.xacro"/> -->
+  <xacro:include filename="$(find xarm_description)/urdf/xarm_device.urdf.xacro"/>
+  <link name="justina_arm_base_link"/>
+  <joint name="body_arm_base_joint" type="fixed">
+    <origin xyz="0 0 0.175" rpy="0 0 0"/>
+    <parent link="body_link"/>
+    <child link="justina_arm_base_link"/>
+  </joint>
 </robot>

File: ros2_ws/src/hardware/justina_description/urdf/justina_base.xacro (robot description, xacro)
@@ -3,7 +3,7 @@
     <!-- Robot Parameters -->
     <xacro:property name="PI" value="3.14159265"/>
-    <xacro:property name="body_length" value="0.5"/>
-    <xacro:property name="body_width" value="0.3"/>
-    <xacro:property name="body_height" value="0.25"/>
+    <xacro:property name="body_length" value="0.45"/>
+    <xacro:property name="body_width" value="0.35"/>
+    <xacro:property name="body_height" value="0.35"/>
     <xacro:property name="body_density" value="7850.0"/> <!-- Steel -->
     <xacro:property name="body_mass" value="${body_density * body_length * body_height * body_width}"/>
@@ -15,4 +15,5 @@
     <xacro:property name="wheel_separation" value="${body_width + wheel_width}"/>
     <xacro:property name="wheel_offset" value="${body_length/2 - wheel_radius}"/>
+    <xacro:property name="wheel_offset_z" value="0.1"/>
     <xacro:property name="wheel_density" value="900"/> <!-- Ruber -->
     <xacro:property name="wheel_mass" value="${wheel_density * PI * wheel_radius * wheel_radius * wheel_width}"/>
@@ -125,5 +126,5 @@
     <!-- Left Wheel Joint -->
     <joint name="left_wheel_joint" type="continuous">
-        <origin xyz="-${wheel_offset} ${wheel_separation/2} -${wheel_radius/2}" rpy="0 0 0"/>
+        <origin xyz="${wheel_offset} ${wheel_separation/2} ${-wheel_radius/2 - wheel_offset_z}" rpy="0 0 0"/>
         <parent link="body_link"/>
         <child link="left_wheel_link"/>
@@ -134,5 +135,5 @@
     <!-- Right Wheel Joint -->
     <joint name="right_wheel_joint" type="continuous">
-        <origin xyz="-${wheel_offset} ${-wheel_separation/2} -${wheel_radius/2}" rpy="0 0 0"/>
+        <origin xyz="${wheel_offset} ${-wheel_separation/2} ${-wheel_radius/2 - wheel_offset_z}" rpy="0 0 0"/>
         <parent link="body_link"/>
         <child link="right_wheel_link"/>
@@ -143,5 +144,5 @@
     <!-- Caster Wheel Joint (fixed) -->
     <joint name="caster_joint" type="fixed">
-        <origin xyz="${caster_offset} 0 -${caster_radius/2}" rpy="0 0 0"/>
+        <origin xyz="${-caster_offset} 0 ${-caster_radius/2 - wheel_offset_z}" rpy="0 0 0"/>
         <parent link="body_link"/>
         <child link="caster_link"/>

Commit message: First working justina_gui. Remove arm from urdf

File: ros2_ws/src/hardware/justina_description/urdf/justina.xacro (robot description, xacro)
@@ -2,5 +2,5 @@
 <robot name="justina" xmlns:xacro="http://www.ros.org/wiki/xacro">
   <xacro:include filename="$(find justina_description)/urdf/justina_base.xacro"/>
-  <xacro:include filename="$(find xarm_description)/urdf/xarm_device.urdf.xacro"/>
+  <!-- <xacro:include filename="$(find xarm_description)/urdf/xarm_device.urdf.xacro"/> -->
   <link name="justina_arm_base_link"/>
   <joint name="body_arm_base_joint" type="fixed">

File: ros2_ws/src/hardware/justina_description/urdf/justina_base.xacro (robot description, xacro)
@@ -37,4 +37,5 @@
     <xacro:property name="max_linear_acceleration" value="10"/>
     <!-- Links -->
+    <link name="base_footprint"/>
     <!-- Body Link -->
     <link name="body_link">
@@ -151,16 +152,21 @@
       </inertial>
    </link>
-    <!-- Joints -->
-    <!-- Left Wheel Joint -->
-    <joint name="left_wheel_joint" type="continuous">
-        <origin xyz="${wheel_offset} ${wheel_separation/2} ${-wheel_radius/2 - wheel_offset_z}" rpy="0 0 0"/>
-        <parent link="body_link"/>
-        <child link="left_wheel_link"/>
-        <axis xyz="0 1 0"/>
-        <limit effort="100" velocity="10.0"/>
-        <dynamics damping="0.1" friction="0.1"/>
-    </joint>
-    <!-- Right Wheel Joint -->
-    <joint name="right_wheel_joint" type="continuous">
+   <!-- Joints -->
+   <joint name="base_to_body" type="fixed">
+     <origin xyz="0 0 ${body_height/2}" rpy="0 0 0"/>
+     <parent link="base_footprint"/>
+     <child link="body_link"/>
+   </joint>
+   <!-- Left Wheel Joint -->
+   <joint name="left_wheel_joint" type="continuous">
+     <origin xyz="${wheel_offset} ${wheel_separation/2} ${-wheel_radius/2 - wheel_offset_z}" rpy="0 0 0"/>
+     <parent link="body_link"/>
+     <child link="left_wheel_link"/>
+     <axis xyz="0 1 0"/>
+     <limit effort="100" velocity="10.0"/>
+     <dynamics damping="0.1" friction="0.1"/>
+   </joint>
+   <!-- Right Wheel Joint -->
+   <joint name="right_wheel_joint" type="continuous">
         <origin xyz="${wheel_offset} ${-wheel_separation/2} ${-wheel_radius/2 - wheel_offset_z}" rpy="0 0 0"/>
         <parent link="body_link"/>
@@ -205,19 +211,22 @@
     <!-- Gazebo Plugins -->
     <gazebo>
-        <plugin filename="gz-sim-diff-drive-system" name="gz::sim::systems::DiffDrive">
-            <right_joint>right_wheel_joint</right_joint>
-            <left_joint>left_wheel_joint</left_joint>
-            <wheel_separation>${wheel_separation}</wheel_separation>
-            <wheel_radius>${wheel_radius}</wheel_radius>
-            <max_linear_acceleration>${max_linear_acceleration}</max_linear_acceleration>
-            <odom_publish_frequency>100</odom_publish_frequency>
-            <topic>cmd_vel</topic>
-            <odom_topic>odom</odom_topic>
-        </plugin>
-        <plugin filename="gz-sim-joint-state-publisher-system" name="gz::sim::systems::JointStatePublisher">
-            <topic>joint_states</topic>
-            <joint_name>right_wheel_joint</joint_name>
-            <joint_name>left_wheel_joint</joint_name>
-        </plugin>
+      <plugin filename="gz-sim-diff-drive-system" name="gz::sim::systems::DiffDrive">
+        <right_joint>right_wheel_joint</right_joint>
+        <left_joint>left_wheel_joint</left_joint>
+        <wheel_separation>${wheel_separation}</wheel_separation>
+        <wheel_radius>${wheel_radius}</wheel_radius>
+        <max_linear_acceleration>${max_linear_acceleration}</max_linear_acceleration>
+        <odom_publish_frequency>20</odom_publish_frequency>
+        <topic>cmd_vel</topic>
+        <tf_topic>tf</tf_topic>
+        <frame_id>/odom</frame_id>
+        <child_frame_id>/base_footprint</child_frame_id>
+        <odom_topic>odom</odom_topic>
+      </plugin>
+      <plugin filename="gz-sim-joint-state-publisher-system" name="gz::sim::systems::JointStatePublisher">
+        <topic>joint_states</topic>
+        <joint_name>right_wheel_joint</joint_name>
+        <joint_name>left_wheel_joint</joint_name>
+      </plugin>
     </gazebo>
     <gazebo reference="laser_link">

Commit message: Add files for geometric features

File: ros2_ws/src/hardware/justina_description/urdf/justina.xacro (robot description, xacro)
@@ -2,10 +2,16 @@
 <robot name="justina" xmlns:xacro="http://www.ros.org/wiki/xacro">
   <xacro:include filename="$(find justina_description)/urdf/justina_base.xacro"/>
+  <xacro:include filename="$(find justina_description)/urdf/justina_upper.xacro"/>
+  <joint name="base_torso_joint" type="fixed">
+    <origin xyz="0.0 0.0 0.525" rpy="0 0 0"/>
+    <parent link="body_link"/>
+    <child link="torso_link"/>
+  </joint>
   <!-- <xacro:include filename="$(find xarm_description)/urdf/xarm_device.urdf.xacro"/> -->
-  <link name="justina_arm_base_link"/>
-  <joint name="body_arm_base_joint" type="fixed">
-    <origin xyz="0 0 0.175" rpy="0 0 0"/>
-    <parent link="body_link"/>
-    <child link="justina_arm_base_link"/>
-  </joint>
+  <!-- <link name="justina_arm_base_link"/> -->
+  <!-- <joint name="body_arm_base_joint" type="fixed"> -->
+  <!--   <origin xyz="0 0 0.175" rpy="0 0 0"/> -->
+  <!--   <parent link="body_link"/> -->
+  <!--   <child link="justina_arm_base_link"/> -->
+  <!-- </joint> -->
 </robot>
