Commit message: Add files for final project

File: ros2_ws/src/hardware/justina_description/urdf/justina_upper.xacro (robot description, xacro)
@@ -53,5 +53,5 @@
     </link>
     <joint name="torso_camera_joint" type="fixed">
-      <origin xyz="0.0 0.0 0.36" rpy="0 0 0"/>
+      <origin xyz="0.0 0.0 0.36" rpy="0 0.8 0"/>
       <parent link="torso_link"/>
       <child link="realsense_link"/>
